Commit message: Check in panda sysid changes for stiffer gains.

File: mani_skill/assets/robots/fr3/fr3_agilex_gripper.urdf (robot description, URDF)
Before this commit: robot fr3_agilex_gripper, 26 links, 25 joints
Joints:
- joint fr3_finger_joint1: limit lower=0 upper=0.05 effort=100 velocity=1 -> lower=0 upper=0.035 effort=100 velocity=1
- joint fr3_finger_joint2: limit lower=0 upper=0.05 effort=100 velocity=1 -> lower=0 upper=0.035 effort=100 velocity=1
- joint fr3_gripper_tcp_joint: origin xyz=0 0 0.19 rpy=0 0 0 -> xyz=0 0 0.12 rpy=0 0 0

Commit message: Stable?

File: mani_skill/assets/robots/fr3/fr3_agilex_gripper.urdf (robot description, URDF)
Before this commit: robot fr3_agilex_gripper, 26 links, 25 joints
Joints:
- joint fr3_gripper_base_joint: origin xyz=0 0 0 rpy=0 0 -0.7853981633974483 -> xyz=0 0 0 rpy=0 0 -2.35619449019

File: mani_skill/assets/robots/fr3/fr3_agilex_gripper_wristcam.urdf (robot description, URDF)
Before this commit: robot fr3_agilex_gripper, 27 links, 26 joints
Joints:
- joint fr3_gripper_base_joint: origin xyz=0 0 0 rpy=0 0 -0.7853981633974483 -> xyz=0 0 0 rpy=0 0 -2.35619449019
